Commit message: gazebo 車輪の追加、動作確認済み

File: src/my_robot_description/urdf/my_robot.urdf (robot description, URDF)
Before this commit: robot my_sim_robot, 1 links, 0 joints
Links:
- added link wheel_fl, mass 0.2; collision cylinder length=0.05 radius=0.1; visual cylinder length=0.05 radius=0.1
- added link wheel_fr, mass 0.2; collision cylinder length=0.05 radius=0.1; visual cylinder length=0.05 radius=0.1
- added link wheel_rl, mass 0.2; collision cylinder length=0.05 radius=0.1; visual cylinder length=0.05 radius=0.1
- added link wheel_rr, mass 0.2; collision cylinder length=0.05 radius=0.1; visual cylinder length=0.05 radius=0.1
Joints:
- added joint wheel_fl_joint: type continuous, parent base_link, child wheel_fl, origin xyz=0.2 0.175 0 rpy=1.5708 0 0, axis 0 0 1
- added joint wheel_fr_joint: type continuous, parent base_link, child wheel_fr, origin xyz=0.2 -0.175 0 rpy=1.5708 0 0, axis 0 0 1
- added joint wheel_rl_joint: type continuous, parent base_link, child wheel_rl, origin xyz=-0.2 0.175 0 rpy=1.5708 0 0, axis 0 0 1
- added joint wheel_rr_joint: type continuous, parent base_link, child wheel_rr, origin xyz=-0.2 -0.175 0 rpy=1.5708 0 0, axis 0 0 1
